File: smokewire/smokewire.kicad_pcb (KiCad board)
At the start: 2 copper layers, 83.8 x 48.3 mm, 15 parts, among them Q1 TIP120, U1 LM358

Commit message: Just added a few more comments on the pcb
Other:
- board text added: "GND"
- board text added: "VOUT"
Changed lines of the file:
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@@
 		(layer "Edge.Cuts")
+	)
+	(gr_text "GND"
+		(at 170.815 120.65 0)
+		(layer "F.SilkS")
+		(effects
+			(font
+				(size 1 1)
+				(thickness 0.15)
+			)
+			(justify left bottom)
+		)
+	)
+	(gr_text "VOUT"
+		(at 152.4 121.92 0)
+		(layer "F.SilkS")
+		(effects
+			(font
+				(size 1 1)
+				(thickness 0.15)
+			)
+			(justify left bottom)
+		)
 	)
 	(gr_text "Ref. Resistance"
@@
 		(layer "F.SilkS")
 		(effects
+			(font
+				(size 1 1)
+				(thickness 0.15)
+			)
+			(justify left bottom)
+		)
+	)
+	(gr_text "GND"
+		(at 111.125 106.045 0)
+		(layer "F.SilkS")
+		(effects
